File: IOTV_id1/1.0/relay.kicad_sch (KiCad schematic)
At the start: 15 parts, among them K1 G3MB202PDC12, K2 G3MB202PDC12, K3 G3MB202PDC12, Q1 S8050, Q2 S8050, Q3 S8050

Commit message: id1 (3x2A) 1.0
Проверка резонит.
Parts:
- R3, R4, R5: value 80om -> 100
Other:
- title: (none) -> IOTV_ID-1 (3x2A)
Changed lines of the file:
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@@
 	(paper "A4")
 	(title_block
+		(title "IOTV_ID-1 (3x2A)")
 		(date "2024-07-29")
+		(rev "1.0")
 		(company "Вербкин М.С.")
 	)
@@
 			)
 		)
-		(property "Value" "80om"
+		(property "Value" "100"
 			(at 80.01 91.44 90)
 			(effects
@@
 			)
 		)
-		(property "Value" "80om"
+		(property "Value" "100"
 			(at 156.21 90.17 90)
 			(effects
@@
 			)
 		)
-		(property "Value" "80om"
+		(property "Value" "100"
 			(at 231.14 88.9 90)
 			(effects
