File: IOTV_id1/1.0/IOTV.kicad_pcb (KiCad board)
At the start: 2 copper layers, 21 parts, among them J1 Screw_Terminal_01x02, J2 Screw_Terminal_01x02, J3 Conn_01x04, J8 UART, Q1 S8050, SW1 RST, SW2 Boot, U1 PQSSR-P_input_3-32VDC_output_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, U3 ESP32-WROOM-E

Commit message: id1 1.0
Parts:
- removed J8: UART, Connector_PinHeader_2.54mm:PinHeader_1x04_P2.54mm_Vertical
- removed U3: ESP32-WROOM-E, PCM_Espressif:ESP32-WROOM-32E
- added C7: C_Generic, Capacitor_THT:C_Rect_L13.0mm_W5.0mm_P10.00mm_FKS3_FKP3_MKS4, F.Cu at (51.0, 167.3)
- added C8: C_Generic, Capacitor_THT:CP_Radial_D8.0mm_P5.00mm, F.Cu at (100.2, 165.4)
- added D1: LED, PCM_Diode_SMD_Handsoldering_AKL:D_0603_1608Metric, F.Cu at (80.1, 85.1)
- added D2: LED, PCM_Diode_SMD_Handsoldering_AKL:D_0603_1608Metric, F.Cu at (80.1, 87.4)
- added D3: LED, PCM_Diode_SMD_Handsoldering_AKL:D_0603_1608Metric, F.Cu at (80.1, 89.7)
- added D4: LED, PCM_Diode_SMD_Handsoldering_AKL:D_0603_1608Metric, F.Cu at (80.1, 82.7)
- added F2: 2, Fuse:Fuseholder_Cylinder-5x20mm_Schurter_0031_8201_Horizontal_Open, F.Cu at (66.5, 156.2)
- added F3: 2, Fuse:Fuseholder_Cylinder-5x20mm_Schurter_0031_8201_Horizontal_Open, F.Cu at (83.5, 156.4)
- added F4: 2, Fuse:Fuseholder_Cylinder-5x20mm_Schurter_0031_8201_Horizontal_Open, F.Cu at (100.7, 156.5)
- added J4: Screw_Terminal_01x02, TerminalBlock_Phoenix:TerminalBlock_Phoenix_MKDS-1,5-2_1x02_P5.00mm_Horizontal, F.Cu at (89.0, 164.8)
- added J_I2C1: Conn_01x04, Connector_PinHeader_2.54mm:PinHeader_1x04_P2.54mm_Vertical, F.Cu at (91.2, 98.2)
- added J_UART1: UART, Connector_PinHeader_2.54mm:PinHeader_1x04_P2.54mm_Vertical, F.Cu at (78.8, 98.2)
- added K1: G3MB202PDC12, g3mb-202:RELAY_G3MB202PDC12, F.Cu at (57.9, 145.4)
- added K2: G3MB202PDC12, g3mb-202:RELAY_G3MB202PDC12, F.Cu at (75.1, 145.6)
- added K3: G3MB202PDC12, g3mb-202:RELAY_G3MB202PDC12, F.Cu at (92.2, 145.7)
- added Q2: S8050, Package_TO_SOT_SMD:SOT-23, B.Cu at (80.3, 126.0)
- added Q3: S8050, Package_TO_SOT_SMD:SOT-23, B.Cu at (85.3, 126.0)
- added R3: 80om, Resistor_SMD:R_1206_3216Metric, F.Cu at (84.0, 85.0)
- added R4: 80om, Resistor_SMD:R_1206_3216Metric, F.Cu at (84.0, 87.4)
- added R5: 80om, Resistor_SMD:R_1206_3216Metric, F.Cu at (84.0, 89.7)
- added R6: 330, Resistor_SMD:R_1206_3216Metric, F.Cu at (84.0, 82.7)
- added U2: AMS1117-3.3, Package_TO_SOT_SMD:SOT-223-3_TabPin2, B.Cu at (77.9, 116.4)
- C5: value C_Generic -> 10uF_0805_25V; footprint Capacitor_THT:C_Rect_L13.0mm_W5.0mm_P10.00mm_FKS3_FKP3_MKS4 -> Capacitor_SMD:C_1206_3216Metric; moved to B.Cu
- C6: value C_Generic -> 10uF_0805_25V; footprint Capacitor_THT:CP_Radial_D8.0mm_P5.00mm -> Capacitor_SMD:C_1206_3216Metric; moved to B.Cu
- FL1: footprint PCM_Inductor_THT_AKL:L_CommonMode_Toroid_Vertical_L19.3mm_W10.8mm_Px6.35mm_Py15.24mm_Bourns_8100 -> PCM_Inductor_THT_AKL:L_CommonMode_Toroid_Vertical_10x13mm
- J3: value Conn_01x04 -> Screw_Terminal_01x02; footprint Connector_PinHeader_2.54mm:PinHeader_1x04_P2.54mm_Vertical -> TerminalBlock_Phoenix:TerminalBlock_Phoenix_MKDS-1,5-2_1x02_P5.00mm_Horizontal
- U1: value PQSSR-P_input_3-32VDC_output_5A_380VAC -> ESP32-WROOM-E; footprint Relay_THT:Relay_NCR_HHG1D-1 -> PCM_Espressif:ESP32-WROOM-32E
- moved RVe1 118.5 mm to (46.9, 160.5)
- moved J1 118.1 mm to (45.6, 149.9), turned to -90 degrees
- moved F1 115.3 mm to (45.5, 144.2), turned to 90 degrees
- moved FL1 111.3 mm to (42.8, 105.9), turned to 0 degrees
- moved J3 88.9 mm to (77.6, 164.8), turned to 0 degrees
- moved J2 83.3 mm to (66.2, 164.8)
- moved U1 76.8 mm to (55.4, 89.7), turned to 90 degrees
- moved C5 72.1 mm to (85.2, 118.9)
- moved Q1 70.4 mm to (75.3, 126.1), turned to 90 degrees
- moved PS1 52.3 mm to (63.9, 113.3)
- moved C4 47.8 mm to (61.3, 93.7), turned to 0 degrees
- moved C3 43.3 mm to (61.3, 89.7), turned to 0 degrees
- moved R1 35.1 mm to (56.6, 86.0), turned to 0 degrees
- moved C2 34.7 mm to (51.7, 89.8), turned to 180 degrees
- moved R2 33.9 mm to (61.2, 86.0), turned to 180 degrees
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Connections:
- net Net-(PS1-AC1) renamed FL1-PS1(AC1)
- net Net-(PS1-AC2) renamed FL1-PS1(AC2)
- C5 pad 1: ~220 -> +5V
- C5 pad 2: SSD-1 -> GND
- F1 pad 1: Net-(J1-Pin_1) -> J1/F1/Relay
- F1 pad 2: ~220 -> J1-FL1(2)
- FL1 pad 2: ~220 -> J1-FL1(2)
- FL1 pad 3: SSD-1 -> ~220V_NC
- J1 pad 1: Net-(J1-Pin_1) -> J1/F1/Relay
- J1 pad 2: SSD-1 -> ~220V_NC
- J2 pad 1: Net-(J1-Pin_1) -> ~220V_NC
- J2 pad 2: SSD-2 -> ~220V_COM_1
- J3 pad 1: GND -> ~220V_NC
- J3 pad 2: +3.3V -> ~220V_COM_2
- PS1 pad 4: +3.3V -> +5V
- Q1 pad 2: ssr+ -> Net-(K1-+)
- Q1 pad 3: +3.3V -> +5V
- RVe1 pad 1: ~220 -> J1-FL1(2)
- RVe1 pad 2: SSD-1 -> ~220V_NC
- U1 pad 1: SSD-2 -> GND
- U1 pad 2: SSD-1 -> +3.3V
- U1 pad 3: GND -> EN
- U1 pad 4: ssr+ -> unconnected-(U1-SENSOR_VP/GPIO36/ADC1_CH0-Pad4)
Routing:
- net GND: track 0.00 -> 176.0 mm, vias 0 -> 2
- net +5V: track 0.00 -> 125.2 mm
- net ~220V_NC: track 0.00 -> 101.4 mm
- net Net-(K1-+): track 0.00 -> 69.8 mm, vias 0 -> 1
- net J1-FL1(2): track 0.00 -> 58.4 mm
- net Net-(K2-+): track 0.00 -> 57.5 mm, vias 0 -> 1
- net SCL: track 0.00 -> 56.6 mm, vias 0 -> 1
- net Net-(K3-+): track 0.00 -> 53.7 mm, vias 0 -> 1
- net J1/F1/Relay: track 0.00 -> 52.9 mm
- net GPIO25: track 0.00 -> 50.2 mm, vias 0 -> 1
- net SDA: track 0.00 -> 49.7 mm, vias 0 -> 1
- net GPIO33: track 0.00 -> 46.2 mm, vias 0 -> 1
- net +3.3V: track 0.00 -> 44.2 mm, vias 0 -> 1
- net GPIO32: track 0.00 -> 42.5 mm, vias 0 -> 1
- net U0RX: track 0.00 -> 38.5 mm, vias 0 -> 1
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- added copper zone on B.Cu, net +3.3V
- added copper zone on F.Cu, net GND
Other:
- board outline added: 72 x 97 mm
- board text added: "- Питание"
- board text added: "- Реле_1"
- board text added: "- Реле_2"
- board text added: "- Реле_3"
- board text added: "GND 3.3 SDA SCL"
- board text added: "GND TX RX 3.3|"

Commit message: id1 (3x2A) 1.0
Проверка резонит.
Parts:
- added G***: LOGO, Symbol:logo_10x10, B.Cu at (154.1, 56.9)
- added J5: PINHD_1x2_Male, Connector_PinHeader_2.54mm:PinHeader_1x02_P2.54mm_Vertical, F.Cu at (169.3, 53.3)
- added J6: PINHD_1x2_Male, Connector_PinHeader_2.54mm:PinHeader_1x02_P2.54mm_Vertical, F.Cu at (169.3, 57.1)
- added J7: PINHD_1x2_Male, Connector_PinHeader_2.54mm:PinHeader_1x02_P2.54mm_Vertical, F.Cu at (169.3, 60.9)
- added REF**: MountingHole_2.5mm_Pad, MountingHole:MountingHole_2.5mm_Pad, F.Cu at (174.8, 116.2)
- added REF**: MountingHole_2.5mm_Pad, MountingHole:MountingHole_2.5mm_Pad, F.Cu at (119.6, 104.0)
- F1: value 0.5 -> 1A
- J_I2C1: value Conn_01x04 -> Conn_01x05; footprint Connector_PinHeader_2.54mm:PinHeader_1x04_P2.54mm_Vertical -> Connector_PinHeader_2.54mm:PinHeader_1x05_P2.54mm_Vertical
- J_UART1: value UART -> Conn_01x05; footprint Connector_PinHeader_2.54mm:PinHeader_1x04_P2.54mm_Vertical -> Connector_PinHeader_2.54mm:PinHeader_1x05_P2.54mm_Vertical
- moved J_I2C1 80.2 mm to (166.0, 69.3)
- moved C2 79.5 mm to (125.8, 60.8)
- moved C6 79.5 mm to (159.2, 87.4)
- moved C7 79.5 mm to (125.1, 138.3)
- moved C8 79.5 mm to (174.3, 136.4)
- moved D1 79.5 mm to (154.2, 56.1)
- moved F1 79.5 mm to (119.6, 115.3)
- moved F2 79.5 mm to (140.6, 127.2)
- moved K1 79.5 mm to (132.0, 116.4)
- moved K2 79.5 mm to (149.2, 116.6)
- moved Q1 79.5 mm to (149.3, 97.1)
- moved Q3 79.5 mm to (159.3, 97.1)
- moved R6 79.5 mm to (158.1, 53.7)
- moved SW1 79.5 mm to (146.9, 64.8)
- moved SW2 79.5 mm to (146.9, 56.1)
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Connections:
- U1 pad 12: unconnected-(U1-ADC2_CH7/GPIO27-Pad12) -> GPIO27
- U1 pad 13: unconnected-(U1-MTMS/GPIO14/ADC2_CH6-Pad13) -> GPIO14
- U1 pad 14: unconnected-(U1-MTDI/GPIO12/ADC2_CH5-Pad14) -> GPIO12
Routing:
- net GPIO27: track 0.00 -> 55.5 mm, vias 0 -> 1
- net GPIO14: track 0.00 -> 50.4 mm
- net GPIO12: track 0.00 -> 45.7 mm
- net +3.3V: track 44.2 -> 24.8 mm
- net +5V: track 125.2 -> 141.5 mm
- net GND: track 176.0 -> 173.3 mm
- net FL1-PS1(AC1): track 24.2 -> 25.8 mm
- net FL1-PS1(AC2): track 16.8 -> 18.3 mm
- net Net-(K3-+): track 53.7 -> 55.1 mm
- net SDA: track 49.7 -> 50.5 mm
- net SCL: track 56.6 -> 57.4 mm
- net Net-(K1-+): track 69.8 -> 70.6 mm
Other:
- outline, holes or cut-outs redrawn
- board text added: "+3.3"
- board text added: "+5V"
- board text added: "BOOT"
- board text added: "EN"
- board text added: "GND"
- board text added: "IO12"
- board text added: "IO14"
- board text added: "IO27"
- board text added: "IOTV ID-1 (3x2A)"
- board text added: "RX"
- board text added: "SCL"
- board text added: "SDA"
- board text added: "TX"
- board text added: "rev. 1.0"
- board text removed: "- Питание"
- board text removed: "- Реле_1"
- board text removed: "- Реле_2"
- board text removed: "- Реле_3"
- board text removed: "GND 3.3 SDA SCL"
- board text removed: "GND TX RX 3.3|"

Commit message: id1 (3x2A) 1.0
png файлы
Parts:
- R3, R4, R5: value 80om -> 100
Changed lines of the file:
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@@
 			(pintype "passive")
 		)
-		(model "${KIPRJMOD}/packages3D/D_0603_1608Metric.wrl"
+		(model "${KICAD6_3DMODEL_DIR}/Diode_SMD.3dshapes/D_0603_1608Metric.wrl"
 			(offset
-				(xyz 0 0 0)
+				(xyz -0.08 0 0)
 			)
 			(scale
@@
 			)
 		)
-		(property "Value" "80om"
+		(property "Value" "100"
 			(at 0 1.82 0)
 			(layer "F.Fab")
@@
 			(pintype "passive")
 		)
-		(model "${KIPRJMOD}/packages3D/D_0603_1608Metric.wrl"
+		(model "${KICAD6_3DMODEL_DIR}/Diode_SMD.3dshapes/D_0603_1608Metric.wrl"
 			(offset
-				(xyz 0 0 0)
+				(xyz -0.08 0 0)
 			)
 			(scale
@@
 			)
 		)
-		(property "Display" "n0,1uF/275VAC"
+		(property "Display" "0,1uF/275VAC"
 			(at 0 0 0)
 			(unlocked yes)
@@
 			(pintype "passive")
 		)
-		(model "${KIPRJMOD}/packages3D/D_0603_1608Metric.wrl"
+		(model "${KICAD6_3DMODEL_DIR}/Diode_SMD.3dshapes/D_0603_1608Metric.wrl"
 			(offset
-				(xyz 0 0 0)
+				(xyz -0.08 0 0)
 			)
 			(scale
@@
 			(pintype "passive")
 		)
-		(model "${KIPRJMOD}/packages3D/D_0603_1608Metric.wrl"
+		(model "${KICAD6_3DMODEL_DIR}/Diode_SMD.3dshapes/D_0603_1608Metric.wrl"
 			(offset
-				(xyz 0 0 0)
+				(xyz -0.08 0 0)
 			)
 			(scale
@@
 			)
 		)
-		(property "Value" "80om"
+		(property "Value" "100"
 			(at 0 1.82 0)
 			(layer "F.Fab")
@@
 			)
 		)
-		(property "Value" "80om"
+		(property "Value" "100"
 			(at 0 1.82 0)
 			(layer "F.Fab")
