File: IOTV_id1/1.0/IOTV.kicad_sch (KiCad schematic)
At the start: 21 parts, among them J1 Screw_Terminal_01x02, J2 Screw_Terminal_01x02, J3 Conn_01x04, J8 UART, Q1 S8050, SW1 RST, SW2 Boot, U1 PQSSR-P_input_3-32VDC_output_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, U3 ESP32-WROOM-E

Commit message: id1 1.0
Parts:
- removed C1, C2, C3, C4: C_Generic, Capacitor_SMD:C_1206_3216Metric, symbol PCM_4ms_Capacitor:C_Generic
- removed J3: Conn_01x04, Connector_PinHeader_2.54mm:PinHeader_1x04_P2.54mm_Vertical, symbol Connector_Generic:Conn_01x04
- removed J8: UART, Connector_PinHeader_2.54mm:PinHeader_1x04_P2.54mm_Vertical, symbol Connector_Generic:Conn_01x04
- removed Q1: S8050, Package_TO_SOT_SMD:SOT-23, symbol Simulation_SPICE:NPN
- removed R1: 10K, Resistor_SMD:R_1206_3216Metric, symbol Device:R
- removed R2: 5K, Resistor_SMD:R_1206_3216Metric, symbol Device:R
- removed SW1: RST, Button_Switch_SMD:SW_SPST_TL3342, symbol Switch:SW_Push
- removed SW2: Boot, Button_Switch_SMD:SW_SPST_TL3342, symbol Switch:SW_Push
- removed U1: PQSSR-P_input_3-32VDC_output_5A_380VAC, Relay_THT:Relay_NCR_HHG1D-1, symbol Relay_SolidState:HHG1D-1
- removed U3: ESP32-WROOM-E, PCM_Espressif:ESP32-WROOM-32E, symbol PCM_Espressif:ESP32-WROOM-E
- added J3, J4: Screw_Terminal_01x02, TerminalBlock_Phoenix:TerminalBlock_Phoenix_MKDS-1,5-2_1x02_P5.00mm_Horizontal, symbol Connector:Screw_Terminal_01x02
- C7: renamed from C5; Display 0,1uF -> n0,1uF/275VAC
- FL1: footprint PCM_Inductor_THT_AKL:L_CommonMode_Toroid_Vertical_L19.3mm_W10.8mm_Px6.35mm_Py15.24mm_Bourns_8100 -> PCM_Inductor_THT_AKL:L_CommonMode_Toroid_Vertical_10x13mm
- renumbered C6 to C8
Connections:
- net J1/F1/Relay: now reaches F1.1, J1.1 (Pin_1)
- net J1/F1/Relay: no longer J2.1 (Pin_1)
- net FL1-PS1(AC1): now reaches FL1.1, PS1.1 (AC1)
- net FL1-PS1(AC2): now reaches FL1.4, PS1.2 (AC2)
- net +3.3V renamed +5V
- net SSD-1 renamed ~220V_NC
- net ~220V_NC: now also J2.1 (Pin_1), J3.1 (Pin_1), J4.1 (Pin_1)
- net SSD-2 renamed ~220V_COM_1
- net ~220 renamed J1-FL1(2)
- new net ~220V_COM_2: J3.2 (Pin_2)
- new net ~220V_COM_3: J4.2 (Pin_2)
- no-connect marks 20 -> 0
Other:
- added sheet esp32 (esp32.kicad_sch)
- added sheet relay (relay.kicad_sch)
- moved on the sheet: C7, C8, F1, FL1, J1, J2, PS1, RVe1

Commit message: id1 (3x2A) 1.0
Проверка резонит.
Parts:
- C7: Display n0,1uF/275VAC -> 0,1uF/275VAC
- F1: value 0.5 -> 1A
Other:
- title: IOTV id-1 -> IOTV_ID-1 (3x2A)
Changed lines of the file:
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@@
 	(paper "A4")
 	(title_block
-		(title "IOTV id-1")
+		(title "IOTV_ID-1 (3x2A)")
 		(date "2024-07-29")
-		(rev "3")
+		(rev "1.0")
 		(company "Вербкин М.С.")
 	)
@@
 			)
 		)
-		(property "Display" "n0,1uF/275VAC"
+		(property "Display" "0,1uF/275VAC"
 			(at 121.412 104.14 0)
 			(effects
@@
 			)
 		)
-		(property "Value" "0.5"
+		(property "Value" "1A"
 			(at 104.14 96.52 90)
 			(effects

Commit message: docs +
Parts:
- added C5, C6: 10uF_0805_25V, Capacitor_SMD:C_1206_3216Metric, symbol PCM_4ms_Capacitor:10uF_0805_25V
- added D4: LED, PCM_Diode_SMD_Handsoldering_AKL:D_0603_1608Metric, symbol PCM_SL_Devices:LED
- added R6: 330, Resistor_SMD:R_1206_3216Metric, symbol Device:R
- added U2: AMS1117-3.3, Package_TO_SOT_SMD:SOT-223-3_TabPin2, symbol Regulator_Linear:AMS1117-3.3
Connections:
- net +5V: now also C5.1, R6.2, U2.3 (VI)
- net GND: now also C5.2, C6.2, D4.1, U2.1 (GND)
- new net: D4.2, R6.1
- new net +3.3V: C6.1, U2.2 (VO)
