File: IOTV_id1/1.0/esp32.kicad_sch (KiCad schematic)
At the start: 16 parts, among them SW1 RST, SW2 Boot, U1 ESP32-WROOM-E, U2 AMS1117-3.3

Commit message: id1 (3x2A) 1.0
Проверка резонит.
Parts:
- removed J_I2C1: Conn_01x04, Connector_PinHeader_2.54mm:PinHeader_1x04_P2.54mm_Vertical, symbol Connector_Generic:Conn_01x04
- removed J_UART1: UART, Connector_PinHeader_2.54mm:PinHeader_1x04_P2.54mm_Vertical, symbol Connector_Generic:Conn_01x04
- added J5, J6, J7: PINHD_1x2_Male, Connector_PinHeader_2.54mm:PinHeader_1x02_P2.54mm_Vertical, symbol PCM_SL_Pin_Headers:PINHD_1x2_Male
- added J_I2C1, J_UART1: Conn_01x05, Connector_PinHeader_2.54mm:PinHeader_1x05_P2.54mm_Vertical, symbol Connector_Generic:Conn_01x05
Connections:
- net +3.3V: now also J_I2C1.2 (Pin_2), J_UART1.4 (Pin_4)
- net +5V: now also J_I2C1.5 (Pin_5), J_UART1.5 (Pin_5)
- net GND: now also J5.2, J6.2, J7.2, J_I2C1.1 (Pin_1), J_UART1.1 (Pin_1)
- net SCL: now also J_I2C1.4 (Pin_4)
- net SDA: now also J_I2C1.3 (Pin_3)
- net U0RX: now also J_UART1.3 (Pin_3)
- net U0TX: now also J_UART1.2 (Pin_2)
- net GPIO27: now reaches U1.12 (ADC2_CH7/GPIO27)
- net GPIO27: now also J7.1
- net GPIO14: now reaches U1.13 (MTMS/GPIO14/ADC2_CH6)
- net GPIO14: now also J6.1
- net GPIO12: now reaches U1.14 (MTDI/GPIO12/ADC2_CH5)
- net GPIO12: now also J5.1
- no-connect marks 18 -> 15
Other:
- title: esp32-wroom-e -> IOTV_ID-1 (3x2A)

Commit message: docs +
Parts:
- removed C5, C6: 10uF_0805_25V, Capacitor_SMD:C_1206_3216Metric, symbol PCM_4ms_Capacitor:10uF_0805_25V
- removed D4: LED, PCM_Diode_SMD_Handsoldering_AKL:D_0603_1608Metric, symbol PCM_SL_Devices:LED
- removed R6: 330, Resistor_SMD:R_1206_3216Metric, symbol Device:R
- removed U2: AMS1117-3.3, Package_TO_SOT_SMD:SOT-223-3_TabPin2, symbol Regulator_Linear:AMS1117-3.3
